Commit message: feat(maze_bot/urdf): update wheel and caster collision geometry, friction, and gazebo plugins

File: maze_bot/urdf/maze_bot.urdf (robot description, URDF)
Before this commit: robot maze_bot, 6 links, 5 joints
Links:
- link camera_link: mass None -> 0.05
- link caster: geometry collision sphere radius=0.0138; visual mesh filename=package://maze_bot/meshes/front_caster.stl
- link wheel_left: geometry collision cylinder length=0.032 radius=0.07; visual mesh filename=package://maze_bot/meshes/wheel_l.stl
- link wheel_right: geometry collision cylinder length=0.032 radius=0.07; visual mesh filename=package://maze_bot/meshes/wheel_r.stl
Joints:
- joint base_joint: origin xyz=0 0 0 rpy=0 0 0 -> xyz=0 0 0.03 rpy=0 0 0
- joint caster_joint: origin xyz=-0.14 -0.007 -0.03 rpy=0.0 0.0 0.0 -> xyz=-0.14 -0.007 -0.0162 rpy=0.0 0.0 0.0
- joint wheel_right_joint: origin xyz=0.09 0.085 0.04   rpy=0 0.0 0.0 -> xyz=0.09 0.085 0.04 rpy=0 0.0 0.0
